Commit message: Update padbot URDF

File: padbot/urdf/padbot_u1.urdf (robot description, URDF)
Before this commit: robot padbot_p1, 8 links, 7 joints
Links:
- added link base_footprint; collision box size=0.001 0.001 0.001; visual box size=0.001 0.001 0.001
- added link raspicam, mass 0.01; collision cylinder length=0.005 radius=0.01; visual cylinder length=0.005 radius=0.01
- link pole: geometry collision cylinder length=0.765 radius=0.03; visual cylinder length=0.765 radius=0.03
Joints:
- added joint footprint_base: type fixed, parent base_footprint, child base_link, origin xyz=0.085 0 0.085 rpy=0 0 0
- added joint raspicam_footprint: type fixed, parent base_footprint, child raspicam, origin xyz=0.15 0 0.885 rpy=0 0 -1.5708
- joint tablet_holder_joint: origin xyz=0 0 0.68 rpy=0 0 0 -> xyz=0 0 0.765 rpy=0 0 0
